File: KiCAD/nano/nano.kicad_pcb (KiCad board)
At the start: 2 copper layers, 69.8 x 49.5 mm, 24 parts, among them J1 Barrel_Jack_Switch, J2 Conn_01x02_Male, J3 Conn_01x02_Male, J4 Conn_01x04_Male, J5 Conn_01x03_Male, K1 SANYOU_SRD_Form_C, K2 SANYOU_SRD_Form_C, P1 Digital, P2 Analog, Q1 S8050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

Commit message: reroute wires
Parts:
- moved R3 28.6 mm to (155.8, 115.6), turned to 0 degrees
- moved Q1 22.3 mm to (151.5, 116.5), turned to 0 degrees
- moved R1 18.5 mm to (155.8, 118.7), turned to 0 degrees
- moved Q2 12.4 mm to (151.5, 111.4), turned to 0 degrees
- moved R2 12.1 mm to (155.8, 113.7)
- moved R4 4.49 mm to (155.8, 110.5)
- moved J4 4.44 mm to (150.5, 101.6)
- moved J5 3.81 mm to (150.5, 97.8)
- moved R5 3.32 mm to (155.8, 127.6), turned to 0 degrees
- moved D1 0.12 mm to (138.8, 116.8), turned to 0 degrees
Routing:
- net Net-(D1-Pad2): track 56.6 -> 27.7 mm, vias 2 -> 0
- net Net-(Q1-Pad2): track 25.0 -> 8.83 mm
- net /Reset: track 0.00 -> 15.2 mm
- net HEATER_RELAY: track 3.60 -> 18.1 mm, vias 0 -> 1
- net Net-(D2-Pad2): track 38.0 -> 26.1 mm, vias 2 -> 0
- net FAN_RELAY: track 11.3 -> 22.9 mm, vias 0 -> 1
- net DHT11: track 27.6 -> 36.9 mm
- net +5V: track 14.2 -> 22.1 mm
- net HEATER_VCC: track 93.7 -> 86.9 mm
- net +12V: track 76.3 -> 71.7 mm
- net CTRL: track 22.5 -> 26.9 mm
- net LCD_I2C_SCL: track 12.7 -> 9.72 mm
- net ICD_I2C_SDA: track 18.3 -> 15.9 mm
- net GND: track 136.5 -> 138.7 mm, vias 1 -> 2
- net Net-(D1-Pad1): track 5.29 -> 6.27 mm
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