File: KiCAD/prototype-board/nano.kicad_pcb (KiCad board)
At the start: 2 copper layers, 25 parts, among them J1 Barrel_Jack_Switch, J2 Conn_01x02_Male, J3 Conn_01x02_Male, J4 Conn_01x04_Male, J5 Conn_01x03_Male, K1 SANYOU_SRD_Form_C, K2 SANYOU_SRD_Form_C, P1 Digital, P2 Analog, Q1 S8050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

Commit message: wires replaned
Parts:
- moved BZ1 50.3 mm to (164.9, 104.3), turned to 0 degrees
- moved SW1 45.0 mm to (196.7, 73.2), turned to 180 degrees
- moved J4 38.1 mm to (154.7, 109.3), turned to 270 degrees
- moved P1 37.5 mm to (159.8, 101.7), turned to 180 degrees
- moved P2 34.5 mm to (144.5, 101.7), turned to 180 degrees
- moved R5 29.6 mm to (177.5, 106.8), turned to 90 degrees
- moved D2 25.2 mm to (190.2, 101.7), turned to 180 degrees
- moved J5 22.5 mm to (164.8, 89.0), turned to 180 degrees
- moved K1 12.1 mm to (195.3, 94.1)
- moved K2 12.1 mm to (177.5, 94.1)
- moved R3 11.4 mm to (154.7, 96.6)
- moved R4 10.5 mm to (149.6, 96.6), turned to 90 degrees
- moved R2 10.2 mm to (149.6, 83.9), turned to 90 degrees
- moved J2 9.55 mm to (169.9, 71.2)
- moved R1 9.16 mm to (154.7, 83.9)
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Routing:
- net BUZZER: track 108.6 -> 17.4 mm
- net +5V: track 13.9 -> 102.0 mm
- net DHT11: track 41.9 -> 5.08 mm
- net +12V: track 74.6 -> 107.7 mm
- net HEATER_RELAY: track 32.6 -> 6.13 mm
- net Net-(D2-Pad1): track 8.86 -> 28.3 mm
- net HEATER_VCC: track 8.21 -> 27.4 mm
- net GND: track 184.8 -> 201.9 mm
- net /Reset: track 12.7 -> 0.00 mm
- net Net-(Q1-Pad2): track 64.4 -> 51.9 mm
- net Net-(D1-Pad2): track 12.5 -> 20.5 mm
- net FAN_VCC: track 11.4 -> 19.0 mm
- net Net-(Q2-Pad2): track 53.1 -> 47.5 mm
- net CTRL: track 51.3 -> 46.3 mm
- net LCD_I2C_SCL: track 19.6 -> 23.9 mm
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Other:
- board text added: "Fan"
- board text added: "Heater"
